Commit message: =

File: assets/formular/formular_car/car.urdf (robot description, URDF)
Before this commit: robot formular_car, 9 links, 8 joints
Links:
- link body: geometry collision mesh filename=./components/body.stl scale=1 1 1; visual mesh filename=./components/body.stl scale=1 1 1
- link steering_fl: mass 1e-5 -> 0.5
- link steering_fr: mass 1e-5 -> 0.5
- link steering_rl: mass 1e-5 -> 0.5
- link steering_rr: mass 1e-5 -> 0.5
- link wheel_fl: geometry collision mesh filename=./components/wheel_FL.stl scale=1 1 1; visual mesh filename=./components/wheel_FL.stl scale=1 1 1
- link wheel_fr: geometry collision mesh filename=./components/wheel_FR.stl scale=1 1 1; visual mesh filename=./components/wheel_FR.stl scale=1 1 1
- link wheel_rl: geometry collision mesh filename=./components/wheel_RL.stl scale=1 1 1; visual mesh filename=./components/wheel_RL.stl scale=1 1 1
- link wheel_rr: geometry collision mesh filename=./components/wheel_RR.stl scale=1 1 1; visual mesh filename=./components/wheel_RR.stl scale=1 1 1

Commit message: ~

File: assets/formular/formular_car/car.urdf (robot description, URDF)
Before this commit: robot formular_car, 9 links, 8 joints
Links:
- link body: mass 600.0 -> 100.0

Commit message: L

File: assets/formular/formular_car/car.urdf (robot description, URDF)
Before this commit: robot formular_car, 9 links, 8 joints
Links:
- link body: mass 100.0 -> 800.0
